Commit message: Change structure

File: src/revolute_joint_examples/urdf/positional_jointed_robot.urdf (robot description, URDF)
Before this commit: robot positional_jointed_robot, 2 links, 1 joints
Joints:
- joint base_to_arm: origin xyz=0.25 0 0.05 rpy=0 0 0 -> xyz=0.25 0 0.2 rpy=0 0 0

Commit message: Can now move in Foxglove

File: src/revolute_joint_examples/urdf/positional_jointed_robot.urdf (robot description, URDF)
Before this commit: robot positional_jointed_robot, 2 links, 1 joints
Joints:
- joint base_to_arm: axis 0 0 1 -> 0 1 0

Commit message: Ok adjust so it makes sense

File: src/revolute_joint_examples/urdf/positional_jointed_robot.urdf (robot description, URDF)
Before this commit: robot positional_jointed_robot, 2 links, 1 joints
Joints:
- joint base_to_arm: origin xyz=0.25 0 0.2 rpy=0 0 0 -> xyz=0.25 0 0.1 rpy=0 1.57 0
