Commit message: Fix spacing

File: src/ackermann_car_example/urdf/car.urdf (robot description, URDF)
Before this commit: robot car, 13 links, 12 joints
Links:
- removed link left_front_shock_mount__column
- removed link left_rear_shock_mount__column
- removed link right_front_shock_mount__column
- removed link right_rear_shock_mount__column
- added link left_front_shock_mount_column, mass 0.0001; collision cylinder length=0.0483 radius=0.002; visual cylinder length=0.0483 radius=0.002
- added link left_rear_shock_mount_column, mass 0.0001; collision cylinder length=0.0483 radius=0.002; visual cylinder length=0.0483 radius=0.002
- added link right_front_shock_mount_column, mass 0.0001; collision cylinder length=0.0483 radius=0.002; visual cylinder length=0.0483 radius=0.002
- added link right_rear_shock_mount_column, mass 0.0001; collision cylinder length=0.0483 radius=0.002; visual cylinder length=0.0483 radius=0.002
Joints:
- removed joint chassis_to_left_front_shock_mount__column_joint
- removed joint chassis_to_left_rear_shock_mount__column_joint
- removed joint chassis_to_right_front_shock_mount__column_joint
- removed joint chassis_to_right_rear_shock_mount__column_joint
- removed joint left_front_axle_to_left_front_shock_mount__column_joint
- removed joint left_rear_axle_to_left_rear_shock_mount__column_joint
- removed joint right_front_axle_to_right_front_shock_mount__column_joint
- removed joint right_rear_axle_to_right_rear_shock_mount__column_joint
- added joint chassis_to_left_front_shock_mount_column_joint: type revolute, parent chassis, child left_front_shock_mount_column, origin xyz=0.125 0.058 -0.018 rpy=0.0 0.0 1.5707963267948966, axis 0. 0. 1., limit lower=-0.5235987755982988 upper=0.5235987755982988 effort=0.1 velocity=0.1
- added joint chassis_to_left_rear_shock_mount_column_joint: type fixed, parent chassis, child left_rear_shock_mount_column, origin xyz=-0.125 0.058 -0.018 rpy=0.0 0.0 1.5707963267948966, axis 1. 0. 0.
- added joint chassis_to_right_front_shock_mount_column_joint: type revolute, parent chassis, child right_front_shock_mount_column, origin xyz=0.125 -0.058 -0.018 rpy=0.0 0.0 -1.5707963267948968, axis 0. 0. 1., limit lower=-0.5235987755982988 upper=0.5235987755982988 effort=0.1 velocity=0.1
- added joint chassis_to_right_rear_shock_mount_column_joint: type fixed, parent chassis, child right_rear_shock_mount_column, origin xyz=-0.125 -0.058 -0.018 rpy=0.0 0.0 -1.5707963267948968, axis 1. 0. 0.
- added joint left_front_axle_to_left_front_shock_mount_column_joint: type fixed, parent left_front_shock_mount_column, child left_front_axle, origin xyz=0.0175 0.0 0.0 rpy=0.0 1.5707963267948966 0.0, axis 0. 1. 0.
- added joint left_rear_axle_to_left_rear_shock_mount_column_joint: type fixed, parent left_rear_shock_mount_column, child left_rear_axle, origin xyz=0.0175 0.0 0.0 rpy=0.0 1.5707963267948966 0.0, axis 0. 1. 0.
- added joint right_front_axle_to_right_front_shock_mount_column_joint: type fixed, parent right_front_shock_mount_column, child right_front_axle, origin xyz=0.0175 0.0 0.0 rpy=0.0 1.5707963267948966 0.0, axis 0. 1. 0.
- added joint right_rear_axle_to_right_rear_shock_mount_column_joint: type fixed, parent right_rear_shock_mount_column, child right_rear_axle, origin xyz=0.0175 0.0 0.0 rpy=0.0 1.5707963267948966 0.0, axis 0. 1. 0.

Commit message: remove left rear controller tempory

File: src/ackermann_car_example/urdf/car.urdf (robot description, URDF)
Before this commit: robot car, 13 links, 12 joints
Links:
- removed link left_front
- removed link left_front_axle
- removed link left_front_shock_mount_column
- removed link right_front
- removed link right_front_axle
- removed link right_front_shock_mount_column
Joints:
- removed joint chassis_to_left_front_shock_mount_column_joint
- removed joint chassis_to_right_front_shock_mount_column_joint
- removed joint left_front_axle_to_left_front_shock_mount_column_joint
- removed joint left_front_to_left_front_axle_joint
- removed joint right_front_axle_to_right_front_shock_mount_column_joint
- removed joint right_front_to_right_front_axle_joint

Commit message: Get at least the car left rear wheel working

File: src/ackermann_car_example/urdf/car.urdf (robot description, URDF)
Before this commit: robot car, 7 links, 6 joints
Links:
- removed link left_rear
- removed link left_rear_axle
- removed link left_rear_shock_mount_column
Joints:
- removed joint chassis_to_left_rear_shock_mount_column_joint
- removed joint left_rear_axle_to_left_rear_shock_mount_column_joint
- removed joint left_rear_to_left_rear_axle_joint
