Commit message: Add axle joint

File: src/ackermann_car_example/urdf/inertia.xacro (robot description, xacro)
@@ -29,3 +29,12 @@
         </inertial>
     </xacro:macro>
+    <!-- Inertia of a solid cylinder. Radius is the radius of the cylinder,
+    and height is its height along the z axis. -->
+    <xacro:macro name="solid_cylinder_inertial" params="radius height mass *origin">
+        <inertial>
+            <!-- <xacro:insert_block name="origin"/> -->
+            <mass value="${mass}"/>
+            <inertia ixx="${(1/12) * mass * (3*radius*radius + height*height)}" ixy="0" ixz="0" iyy="${(1/12) * mass * (3*radius*radius + height*height)}" iyz="0" izz="${(1/2) * mass* radius*radius}" />
+        </inertial>
+    </xacro:macro>
 </robot>

File: src/ackermann_car_example/urdf/wheel.xacro (robot description, xacro)
@@ -1,4 +1,6 @@
 <?xml version="1.0"?>
 <robot xmlns:xacro="http://www.ros.org/wiki/xacro">
+    <!-- Import the other macros -->
+    <xacro:include filename="inertia.xacro" />
     <xacro:macro name="wheel" params="id props">
         <xacro:property name="width" value="${props['width_m']}" />
@@ -17,4 +19,7 @@
                 </geometry>
             </collision>
+            <!-- <xacro:solid_cylinder_inertial radius="${radius}" height="${width}" mass="{mass_kg}">
+                <origin xyz="0 0 0" rpy="0 0 0"/>
+            </xacro:solid_cylinder_inertial> -->
             <inertial>
                 <mass value="${mass_kg}"/>
@@ -23,5 +28,5 @@
         </link>
         <gazebo reference="${id}">
-            <material>Gazebo/Black</material>
+            <material>Gazebo/Grey</material>
         </gazebo>
     </xacro:macro>
