Commit message: Change to xacro file

File: src/ackermann_car_example/urdf/car.xacro (robot description, xacro)
@@ -1,4 +1,24 @@
 <?xml version='1.0' encoding='UTF-8'?>
-<robot name="car">
+<robot xmlns:xacro="http://www.ros.org/wiki/xacro" name="car">
+    <link name="chassis">
+        <inertial>
+            <origin xyz="0.0 0.0 0.0" rpy="0.0 -0.0 0.0"/>
+            <mass value="1.7827"/>
+            <inertia ixx="0.0043741515666666664" ixy="0.0" ixz="0.0" iyy="0.022022881566666663" iyz="0.0" izz="0.025254916666666665"/>
+        </inertial>
+        <visual>
+            <geometry>
+                <box size="0.38  0.16  0.062"/>
+            </geometry>
+            <material name="chassis_color"/>
+            <origin xyz="0.0 0.0 0.0" rpy="0.0 -0.0 0.0"/>
+        </visual>
+        <collision name="chassis_collision">
+            <geometry>
+                <box size="0.38  0.16  0.062"/>
+            </geometry>
+            <origin xyz="0.0 0.0 0.0" rpy="0.0 -0.0 0.0"/>
+        </collision>
+    </link>
     <link name="right_rear">
         <inertial>
@@ -60,24 +80,4 @@
         </collision>
     </link>
-    <link name="chassis">
-        <inertial>
-            <origin xyz="0.0 0.0 0.0" rpy="0.0 -0.0 0.0"/>
-            <mass value="1.7827"/>
-            <inertia ixx="0.0043741515666666664" ixy="0.0" ixz="0.0" iyy="0.022022881566666663" iyz="0.0" izz="0.025254916666666665"/>
-        </inertial>
-        <visual>
-            <geometry>
-                <box size="0.38  0.16  0.062"/>
-            </geometry>
-            <material name="chassis_color"/>
-            <origin xyz="0.0 0.0 0.0" rpy="0.0 -0.0 0.0"/>
-        </visual>
-        <collision name="chassis_collision">
-            <geometry>
-                <box size="0.38  0.16  0.062"/>
-            </geometry>
-            <origin xyz="0.0 0.0 0.0" rpy="0.0 -0.0 0.0"/>
-        </collision>
-    </link>
     <joint name="chassis_to_right_rear_shock_mount_column_joint" type="fixed">
         <parent link="chassis"/>

Commit message: Restart from other example

File: src/ackermann_car_example/urdf/car.xacro (robot description, xacro)
@@ -1,119 +1,55 @@
-<?xml version='1.0' encoding='UTF-8'?>
-<robot xmlns:xacro="http://www.ros.org/wiki/xacro" name="car">
-    <link name="chassis">
-        <inertial>
-            <origin xyz="0.0 0.0 0.0" rpy="0.0 -0.0 0.0"/>
-            <mass value="1.7827"/>
-            <inertia ixx="0.0043741515666666664" ixy="0.0" ixz="0.0" iyy="0.022022881566666663" iyz="0.0" izz="0.025254916666666665"/>
-        </inertial>
+<?xml version="1.0"?>
+<robot name="car"
+    xmlns:xacro="http://www.ros.org/wiki/xacro">
+    <!-- Import the wheel macro -->
+    <xacro:include filename="wheel.xacro" />
+    <!-- Define robot parameters -->
+    <xacro:property name="body_length" value="0.5" />
+    <xacro:property name="body_width" value="0.3" />
+    <xacro:property name="body_height" value="0.1" />
+    <xacro:property name="body_mass" value="5.0" />
+    <xacro:property name="wheel_radius" value="0.1" />
+    <xacro:property name="wheel_width" value="0.05" />
+    <xacro:property name="wheel_mass" value="1.0" />
+    <!-- Robot body -->
+    <link name="base_link">
         <visual>
             <geometry>
-                <box size="0.38  0.16  0.062"/>
+                <box size="${body_length} ${body_width} ${body_height}"/>
             </geometry>
-            <material name="chassis_color"/>
-            <origin xyz="0.0 0.0 0.0" rpy="0.0 -0.0 0.0"/>
+            <material name="blue">
+                <color rgba="0 0 0.8 1"/>
+            </material>
         </visual>
-        <collision name="chassis_collision">
+        <collision>
             <geometry>
-                <box size="0.38  0.16  0.062"/>
+                <box size="${body_length} ${body_width} ${body_height}"/>
             </geometry>
-            <origin xyz="0.0 0.0 0.0" rpy="0.0 -0.0 0.0"/>
         </collision>
+        <inertial>
+            <mass value="${body_mass}"/>
+            <inertia ixx="${(1/12) * body_mass * (body_width*body_width + body_height*body_height)}" ixy="0" ixz="0" iyy="${(1/12) * body_mass * (body_length*body_length + body_height*body_height)}" iyz="0" izz="${(1/12) * body_mass * (body_length*body_length + body_width*body_width)}" />
+        </inertial>
     </link>
-    <link name="right_rear">
-        <inertial>
-            <origin xyz="0.0 0.0 0.0" rpy="0.0 -0.0 0.0"/>
-            <mass value="0.0282"/>
-            <inertia ixx="6.3044624999999994e-06" ixy="0.0" ixz="0.0" iyy="6.3044624999999994e-06" iyz="0.0" izz="9.901724999999999e-06"/>
-        </inertial>
-        <visual name="&lt;urdfpy.urdf.Material object at 0x7f70a765bc10&gt;">
-            <geometry>
-                <cylinder radius="0.0265" length="0.024"/>
-            </geometry>
-            <origin xyz="0.0 0.0 0.0" rpy="0.0 -0.0 0.0"/>
-        </visual>
-        <collision name="wheel_collision">
-            <geometry>
-                <cylinder radius="0.0265" length="0.024"/>
-            </geometry>
-            <origin xyz="0.0 0.0 0.0" rpy="0.0 -0.0 0.0"/>
-        </collision>
-    </link>
-    <link name="right_rear_axle">
-        <inertial>
-            <origin xyz="0.0 0.0 0.0" rpy="0.0 -0.0 0.0"/>
-            <mass value="0.0001"/>
-            <inertia ixx="1.0277223333333336e-08" ixy="0.0" ixz="0.0" iyy="1.0277223333333336e-08" iyz="0.0" izz="1.3778000000000001e-10"/>
-        </inertial>
-        <visual>
-            <geometry>
-                <cylinder radius="0.00166" length="0.035"/>
-            </geometry>
-            <material name="axle_color"/>
-            <origin xyz="0.0 0.0 0.0" rpy="0.0 -0.0 0.0"/>
-        </visual>
-        <collision name="right_rear_axle_collision">
-            <geometry>
-                <cylinder radius="0.00166" length="0.035"/>
-            </geometry>
-            <origin xyz="0.0 0.0 0.0" rpy="0.0 -0.0 0.0"/>
-        </collision>
-    </link>
-    <link name="right_rear_shock_mount_column">
-        <inertial>
-            <origin xyz="0.0 0.0 0.0" rpy="0.0 -0.0 0.0"/>
-            <mass value="0.0001"/>
-            <inertia ixx="1.9540750000000002e-08" ixy="0.0" ixz="0.0" iyy="1.9540750000000002e-08" iyz="0.0" izz="2e-10"/>
-        </inertial>
-        <visual>
-            <geometry>
-                <cylinder radius="0.002" length="0.0483"/>
-            </geometry>
-            <material name="shock_mount_column_color"/>
-            <origin xyz="0.0 0.0 0.0" rpy="0.0 -0.0 0.0"/>
-        </visual>
-        <collision name="right_rear_shock_mount_column_collision">
-            <geometry>
-                <cylinder radius="0.002" length="0.0483"/>
-            </geometry>
-            <origin xyz="0.0 0.0 0.0" rpy="0.0 -0.0 0.0"/>
-        </collision>
-    </link>
-    <joint name="chassis_to_right_rear_shock_mount_column_joint" type="fixed">
-        <parent link="chassis"/>
-        <child link="right_rear_shock_mount_column"/>
-        <axis xyz="1. 0. 0."/>
-        <origin xyz="-0.125 -0.058 -0.018" rpy="0.0 0.0 -1.5707963267948968"/>
+    <!-- Use the wheel macro to create a wheel -->
+    <xacro:wheel id="wheel" radius="${wheel_radius}" width="${wheel_width}" mass_kg="${wheel_mass}" />
+    <!-- Joint connecting the body to the wheel -->
+    <joint name="right_rear_to_right_rear_axle_joint" type="continuous">
+        <parent link="base_link"/>
+        <child link="wheel"/>
+        <origin xyz="${body_length/2} 0 ${-body_height/2}" rpy="${pi/2} 0 0"/>
+        <axis xyz="0 0 1"/>
     </joint>
-    <joint name="right_rear_to_right_rear_axle_joint" type="continuous">
-        <parent link="right_rear_axle"/>
-        <child link="right_rear"/>
-        <axis xyz="0. 0. 1."/>
-        <origin xyz="0.0 0.0 0.004500000000000001" rpy="0.0 0.0 0.0"/>
-    </joint>
-    <joint name="right_rear_axle_to_right_rear_shock_mount_column_joint" type="fixed">
-        <parent link="right_rear_shock_mount_column"/>
-        <child link="right_rear_axle"/>
-        <axis xyz="0. 1. 0."/>
-        <origin xyz="0.0175 0.0 0.0" rpy="0.0 1.5707963267948966 0.0"/>
-    </joint>
-    <transmission name="right_rear_to_right_rear_axle_joint_transmission">
+    <!-- Transmission for the wheel joint -->
+    <transmission name="wheel_trans">
         <type>transmission_interface/SimpleTransmission</type>
         <joint name="right_rear_to_right_rear_axle_joint">
             <hardwareInterface>hardware_interface/VelocityJointInterface</hardwareInterface>
         </joint>
-        <actuator name="right_rear_to_right_rear_axle_joint_actuator">
+        <actuator name="wheel_motor">
+            <hardwareInterface>hardware_interface/VelocityJointInterface</hardwareInterface>
             <mechanicalReduction>1</mechanicalReduction>
         </actuator>
     </transmission>
-    <material name="axle_color">
-        <color rgba="0.5 0.5 0.5 1. "/>
-    </material>
-    <material name="shock_mount_column_color">
-        <color rgba="0.5 0.5 0.5 1. "/>
-    </material>
-    <material name="chassis_color">
-        <color rgba="0. 0. 0. 1."/>
-    </material>
     <!-- Gazebo plugin for ROS Control -->
     <gazebo>
@@ -124,9 +60,3 @@
         </plugin>
     </gazebo>
-    <gazebo reference="right_rear">
-        <material>Gazebo/Black</material>
-    </gazebo>
-    <gazebo reference="chassis">
-        <material>Gazebo/White</material>
-    </gazebo>
 </robot>

Commit message: Fix spelling

File: src/ackermann_car_example/urdf/car.xacro (robot description, xacro)
@@ -2,54 +2,38 @@
 <robot name="car"
     xmlns:xacro="http://www.ros.org/wiki/xacro">
-    <!-- Import the wheel macro -->
+    <!-- Import parameters from the config files -->
+    <xacro:property name="yaml_file" value="$(find ackermann_car_example)/config/car.yml" />
+    <xacro:property name="props" value="${xacro.load_yaml(yaml_file)}" />
+    <xacro:property name="car" value="${props['car']}" />
+    <xacro:property name="chassis" value="${car['chassis']}" />
+    <xacro:property name="wheel" value="${car['wheel']}" />
+    <xacro:property name="tire" value="${car['tire']}" />
+    <xacro:property name="axle" value="${car['axle']}" />
+    <xacro:property name="steering_column" value="${car['steering_column']}" />
+    <xacro:property name="lidar" value="${car['lidar']}" />
+    <xacro:property name="mounts" value="${car['mounts']}" />
+    <!-- Import the other macros -->
     <xacro:include filename="wheel.xacro" />
-    <!-- Define robot parameters -->
-    <xacro:property name="body_length" value="0.5" />
-    <xacro:property name="body_width" value="0.3" />
-    <xacro:property name="body_height" value="0.1" />
-    <xacro:property name="body_mass" value="5.0" />
-    <xacro:property name="wheel_radius" value="0.1" />
-    <xacro:property name="wheel_width" value="0.05" />
-    <xacro:property name="wheel_mass" value="1.0" />
+    <!-- Define IDS -->
+    <xacro:property name="robot_id" value="car" />
+    <xacro:property name="right_rear_id" value="right_rear" />
+    <xacro:property name="left_rear_id" value="left_rear" />
+    <xacro:property name="right_front_id" value="right_front" />
+    <xacro:property name="left_front_id" value="right_front" />
     <!-- Robot body -->
     <link name="base_link">
-        <visual>
-            <geometry>
-                <box size="${body_length} ${body_width} ${body_height}"/>
-            </geometry>
-            <material name="blue">
-                <color rgba="0 0 0.8 1"/>
-            </material>
-        </visual>
-        <collision>
-            <geometry>
-                <box size="${body_length} ${body_width} ${body_height}"/>
-            </geometry>
-        </collision>
         <inertial>
-            <mass value="${body_mass}"/>
-            <inertia ixx="${(1/12) * body_mass * (body_width*body_width + body_height*body_height)}" ixy="0" ixz="0" iyy="${(1/12) * body_mass * (body_length*body_length + body_height*body_height)}" iyz="0" izz="${(1/12) * body_mass * (body_length*body_length + body_width*body_width)}" />
+            <mass value="0.001"/>
+            <inertia ixx="0.0001" ixy="0" ixz="0" iyy="0.0001" iyz="0" izz="0.0001"/>
         </inertial>
     </link>
-    <!-- Use the wheel macro to create a wheel -->
-    <xacro:wheel id="wheel" radius="${wheel_radius}" width="${wheel_width}" mass_kg="${wheel_mass}" />
-    <!-- Joint connecting the body to the wheel -->
-    <joint name="right_rear_to_right_rear_axle_joint" type="continuous">
-        <parent link="base_link"/>
-        <child link="wheel"/>
-        <origin xyz="${body_length/2} 0 ${-body_height/2}" rpy="${pi/2} 0 0"/>
+    <joint name="base_to_wheel" type="fixed">
+        <parent link="base_link" />
+        <child link="${right_rear_id}" />
+        <origin xyz="${chassis.length_m/2 - chassis.wheel_x_offset_from_edge_m} 0 ${chassis.height_m/2}" />
         <axis xyz="0 0 1"/>
     </joint>
-    <!-- Transmission for the wheel joint -->
-    <transmission name="wheel_trans">
-        <type>transmission_interface/SimpleTransmission</type>
-        <joint name="right_rear_to_right_rear_axle_joint">
-            <hardwareInterface>hardware_interface/VelocityJointInterface</hardwareInterface>
-        </joint>
-        <actuator name="wheel_motor">
-            <hardwareInterface>hardware_interface/VelocityJointInterface</hardwareInterface>
-            <mechanicalReduction>1</mechanicalReduction>
-        </actuator>
-    </transmission>
+    <!-- Use the wheel macro to create a wheel -->
+    <xacro:wheel id="${right_rear_id}" props="${wheel}" />
     <!-- Gazebo plugin for ROS Control -->
     <gazebo>

File: src/ackermann_car_example/urdf/wheel.xacro (robot description, xacro)
@@ -1,5 +1,8 @@
 <?xml version="1.0"?>
 <robot xmlns:xacro="http://www.ros.org/wiki/xacro">
-    <xacro:macro name="wheel" params="id radius width mass_kg">
+    <xacro:macro name="wheel" params="id props">
+        <xacro:property name="width" value="${props['width_m']}" />
+        <xacro:property name="mass_kg" value="${props['mass_kg']}" />
+        <xacro:property name="radius" value="${props['diameter_m'] / 2}" />
         <link name="${id}">
             <visual>

Commit message: Fix positional config

File: src/ackermann_car_example/urdf/car.xacro (robot description, xacro)
@@ -1,4 +1,30 @@
 <?xml version='1.0' encoding='UTF-8'?>
 <robot xmlns:xacro="http://www.ros.org/wiki/xacro" name="car">
+    <link name="base_link">
+        <inertial>
+            <origin xyz="0.0 0.0 0.0" rpy="0.0 -0.0 0.0"/>
+            <mass value="1.7827"/>
+            <inertia ixx="0.0043741515666666664" ixy="0.0" ixz="0.0" iyy="0.022022881566666663" iyz="0.0" izz="0.025254916666666665"/>
+        </inertial>
+        <visual>
+            <geometry>
+                <box size="0.01  0.010  0.001"/>
+            </geometry>
+            <material name="chassis_color"/>
+            <origin xyz="0.0 0.0 0.0" rpy="0.0 -0.0 0.0"/>
+        </visual>
+        <collision name="base_link_collision">
+            <geometry>
+                <box size="0.01  0.010  0.001"/>
+            </geometry>
+            <origin xyz="0.0 0.0 0.0" rpy="0.0 -0.0 0.0"/>
+        </collision>
+    </link>
+    <joint name="base_to_chassis_joint" type="fixed">
+        <parent link="base_link"/>
+        <child link="chassis"/>
+        <axis xyz="0. 1. 0."/>
+        <origin xyz="0.0 0.0 0.0" rpy="0.0 0.0 0.0"/>
+    </joint>
     <link name="chassis">
         <inertial>
@@ -27,5 +53,5 @@
             <inertia ixx="6.3044624999999994e-06" ixy="0.0" ixz="0.0" iyy="6.3044624999999994e-06" iyz="0.0" izz="9.901724999999999e-06"/>
         </inertial>
-        <visual name="&lt;urdfpy.urdf.Material object at 0x7f70a765bc10&gt;">
+        <visual>
             <geometry>
                 <cylinder radius="0.0265" length="0.024"/>
@@ -86,9 +112,11 @@
         <origin xyz="-0.125 -0.058 -0.018" rpy="0.0 0.0 -1.5707963267948968"/>
     </joint>
-    <joint name="right_rear_to_right_rear_axle_joint" type="continuous">
+    <joint name="right_rear_to_right_rear_axle_joint" type="revolute">
         <parent link="right_rear_axle"/>
         <child link="right_rear"/>
         <axis xyz="0. 0. 1."/>
         <origin xyz="0.0 0.0 0.004500000000000001" rpy="0.0 0.0 0.0"/>
+        <limit lower="-1.57" upper="1.57" effort="100" velocity="1"/>
+        <dynamics damping="0.1" friction="0.1"/>
     </joint>
     <joint name="right_rear_axle_to_right_rear_shock_mount_column_joint" type="fixed">
@@ -98,4 +126,14 @@
         <origin xyz="0.0175 0.0 0.0" rpy="0.0 1.5707963267948966 0.0"/>
     </joint>
+    <transmission name="right_rear_axle_to_right_rear_shock_mount_column_joint_transmission">
+        <type>transmission_interface/SimpleTransmission</type>
+        <joint name="right_rear_axle_to_right_rear_shock_mount_column_joint">
+            <hardwareInterface>hardware_interface/VelocityJointInterface</hardwareInterface>
+        </joint>
+        <actuator name="right_rear_axle_to_right_rear_shock_mount_column_joint_actuator">
+            <hardwareInterface>hardware_interface/VelocityJointInterface</hardwareInterface>
+            <mechanicalReduction>1</mechanicalReduction>
+        </actuator>
+    </transmission>
     <transmission name="right_rear_to_right_rear_axle_joint_transmission">
         <type>transmission_interface/SimpleTransmission</type>
@@ -104,4 +142,5 @@
         </joint>
         <actuator name="right_rear_to_right_rear_axle_joint_actuator">
+            <hardwareInterface>hardware_interface/VelocityJointInterface</hardwareInterface>
             <mechanicalReduction>1</mechanicalReduction>
         </actuator>
